File: source/source.kicad_pcb (KiCad board)
At the start: 4 copper layers, 102.3 x 70 mm, 61 parts, among them J1 USB_C_Receptacle_USB2.0_14P, J2 Conn_02x13_Odd_Even, J3 Conn_02x13_Odd_Even, U1 ESP32-S3-WROOM-1, U3 AP2112K-1.2, U4 USBLC6-2SC6, U5 MIC29302WU

Commit message: EEE
Parts:
- moved 5V2 2.81 mm to (270.2, 98.1)
- moved JP1 1.20 mm to (174.1, 102.9)
- moved D16 0.45 mm to (243.5, 117.5)
- moved D12 0.19 mm to (259.1, 101.6)
- moved D10 0.18 mm to (251.0, 94.2)
- moved D5 0.17 mm to (228.7, 101.1)
- moved D7 0.16 mm to (236.6, 93.7)
- moved D13 0.13 mm to (255.9, 105.4)
- moved 5V1 0.10 mm to (177.4, 98.1)
- moved D2 0.07 mm to (240.1, 113.2)
- moved D4 0.07 mm to (232.0, 105.1)
- moved D15 0.06 mm to (247.8, 113.6)
Routing:
- net +1V2: track 70.3 -> 75.1 mm
- net +5V: track 112.8 -> 115.8 mm
- net Net-(J2-Pin_10): track 39.2 -> 40.7 mm
- net Net-(D3-DOUT): track 10.5 -> 11.9 mm
- net Net-(D10-DIN): track 10.5 -> 11.1 mm
Other:
- board size 102.3 x 70 mm -> 102.3 x 71.6 mm

Commit message: e
Parts:
- removed JP1: Jumper_3_Bridged12, Connector_PinHeader_2.54mm:PinHeader_1x03_P2.54mm_Vertical
- added J4: Conn_01x13, Connector_PinHeader_2.54mm:PinHeader_1x13_P2.54mm_Vertical, F.Cu at (267.0, 64.1)
- added J5: Conn_01x13, Connector_PinHeader_2.54mm:PinHeader_1x13_P2.54mm_Vertical, F.Cu at (270.1, 94.2)
- added J6: Conn_01x03, Connector_PinHeader_2.54mm:PinHeader_1x03_P2.54mm_Vertical, F.Cu at (174.3, 102.9)
- J2, J3: value Conn_02x13_Odd_Even -> Conn_01x13; footprint Connector_PinHeader_2.54mm:PinHeader_2x13_P2.54mm_Vertical -> Connector_PinHeader_2.54mm:PinHeader_1x13_P2.54mm_Vertical
- moved J3 90.9 mm to (176.8, 64.1)
- moved J2 0.35 mm to (173.9, 64.0)
- moved 5V2 0.20 mm to (270.0, 98.1)
- renumbered buzzer to BZ1
Connections:
- J2 pad 10: Net-(J2-Pin_10) -> 12
- J2 pad 11: 7 -> 13
- J2 pad 12: Net-(J2-Pin_10) -> 14
- J2 pad 13: 9 -> 15
- J2 pad 2: Net-(J2-Pin_10) -> 2
- J2 pad 3: 2 -> 3
- J2 pad 4: Net-(J2-Pin_10) -> 5
- J2 pad 5: 3 -> 6
- J2 pad 6: Net-(J2-Pin_10) -> 7
- J2 pad 7: 5 -> 9
- J2 pad 8: Net-(J2-Pin_10) -> 10
- J2 pad 9: 6 -> 11
- J3 pad 1: GND -> Net-(J3-Pin_1)
- J3 pad 10: 21 -> Net-(J3-Pin_1)
- J3 pad 11: GND -> Net-(J3-Pin_1)
- J3 pad 12: 38 -> Net-(J3-Pin_1)
- J3 pad 13: GND -> Net-(J3-Pin_1)
- J3 pad 2: DTX -> Net-(J3-Pin_1)
- J3 pad 3: GND -> Net-(J3-Pin_1)
- J3 pad 4: DRX -> Net-(J3-Pin_1)
- J3 pad 5: GND -> Net-(J3-Pin_1)
- J3 pad 6: SCL -> Net-(J3-Pin_1)
- J3 pad 7: GND -> Net-(J3-Pin_1)
- J3 pad 8: SDA -> Net-(J3-Pin_1)
- J3 pad 9: GND -> Net-(J3-Pin_1)
Routing:
- net Net-(J3-Pin_1): track 0.00 -> 40.7 mm
- net Net-(J2-Pin_10): track 40.7 -> 0.00 mm
- net GND: track 56.1 -> 86.9 mm
- net 4: track 72.8 -> 74.7 mm
- net +1V2: track 75.1 -> 73.8 mm
- net 8: track 59.8 -> 60.8 mm
- net 13: track 56.3 -> 55.4 mm
- net 41: track 44.9 -> 45.6 mm
Other:
- board size 102.3 x 71.6 mm -> 99.6 x 71.6 mm
