File: source/source.kicad_sch (KiCad schematic)
At the start: 61 parts, among them J1 USB_C_Receptacle_USB2.0_14P, J2 Conn_02x13_Odd_Even, J3 Conn_02x13_Odd_Even, SW1 SW_Push, SW2 SW_Push, U1 ESP32-S3-WROOM-1, U3 AP2112K-1.2, U4 USBLC6-2SC6, U5 MIC29302WU

Commit message: e
Parts:
- removed J2, J3: Conn_02x13_Odd_Even, Connector_PinHeader_2.54mm:PinHeader_2x13_P2.54mm_Vertical, symbol Connector_Generic:Conn_02x13_Odd_Even
- removed JP1: Jumper_3_Bridged12, Connector_PinHeader_2.54mm:PinHeader_1x03_P2.54mm_Vertical, symbol Jumper:Jumper_3_Bridged12
- added J2, J3, J4, J5: Conn_01x13, Connector_PinHeader_2.54mm:PinHeader_1x13_P2.54mm_Vertical, symbol Connector_Generic:Conn_01x13
- added J6: Conn_01x03, Connector_PinHeader_2.54mm:PinHeader_1x03_P2.54mm_Vertical, symbol Connector_Generic:Conn_01x03
Connections:
- net +1V2: now also J6.1 (Pin_1)
- net +3V3: now also J6.3 (Pin_3)
- net 1: now also J2.1 (Pin_1)
- net 10: now also J2.8 (Pin_8)
- net 11: now also J2.9 (Pin_9)
- net 12: now also J2.10 (Pin_10)
- net 13: now also J2.11 (Pin_11)
- net 14: now also J2.12 (Pin_12)
- net 15: now also J2.13 (Pin_13)
- net 2: now also J2.2 (Pin_2)
- net 21: now also J5.9 (Pin_9)
- net 3: now also J2.3 (Pin_3)
- net 38: now also J5.8 (Pin_8)
- net 39: now also J5.7 (Pin_7)
- net 40: now also J5.6 (Pin_6)
- net 41: now also J5.5 (Pin_5)
- net 42: now also J5.4 (Pin_4)
- net 45: now also J5.3 (Pin_3)
- net 46: now also J5.2 (Pin_2)
- net 47: now also J5.1 (Pin_1)
- net 5: now also J2.4 (Pin_4)
- net 6: now also J2.5 (Pin_5)
- net 7: now also J2.6 (Pin_6)
- net 9: now also J2.7 (Pin_7)
- net DRX: now also J5.12 (Pin_12)
- net DTX: now also J5.13 (Pin_13)
- net GND: now also J4.1 (Pin_1), J4.10 (Pin_10), J4.11 (Pin_11), J4.12 (Pin_12), J4.13 (Pin_13), J4.2 (Pin_2), J4.3 (Pin_3), J4.4 (Pin_4), J4.5 (Pin_5), J4.6 (Pin_6), J4.7 (Pin_7), J4.8 (Pin_8), J4.9 (Pin_9)
- net SCL: now also J5.11 (Pin_11)
- net SDA: now also J5.10 (Pin_10)
- new net: J3.1 (Pin_1), J3.10 (Pin_10), J3.11 (Pin_11), J3.12 (Pin_12), J3.13 (Pin_13), J3.2 (Pin_2), J3.3 (Pin_3), J3.4 (Pin_4), J3.5 (Pin_5), J3.6 (Pin_6), J3.7 (Pin_7), J3.8 (Pin_8), J3.9 (Pin_9), J6.2 (Pin_2)
